File: piccolo/piccolo.kicad_pcb (KiCad board)
At the start: 2 copper layers, 136.5 x 20.6 mm, 17 parts, among them SW1 SW_Push, SW2 Rotary_Encoder_Switch, U1 ProMicro

Commit message: First prototype of piccolo ready for production
Parts:
- added GND: SolderJumper_2_Open, Keyboard parts:SOLDER_JUMPER_2, B.Cu at (81.0, 45.3)
- added SCL: SolderJumper_2_Open, Keyboard parts:SOLDER_JUMPER_2, B.Cu at (81.0, 50.4)
- added SDA: SolderJumper_2_Open, Keyboard parts:SOLDER_JUMPER_2, B.Cu at (81.0, 53.0)
- added VCC: SolderJumper_2_Open, Keyboard parts:SOLDER_JUMPER_2, B.Cu at (81.0, 47.9)
- D1, D2, D3, D4, D5: footprint kbd:D3_TH_SMD -> Keebio-Parts:Diode-Hybrid-Back
- Reset: renamed from SW1; value SW_Push -> Reset; moved to B.Cu
- moved Reset 4.95 mm to (179.8, 51.6), turned to 90 degrees
- moved ENC1 0.95 mm to (173.0, 48.3)
- moved D5 0.38 mm to (162.3, 50.8), turned to 270 degrees
- turned D1 to 180 degrees
- turned D2 to 180 degrees
- turned D3 to 180 degrees
- turned D4 to 180 degrees
- renumbered SW2 to ENC1
Connections:
- ENC1 pad S1: Net-(D3-Pad2) -> Net-(D5-Pad2)
- ENC1 pad S2: col2 -> col1
- OL1 pad 1: SDA -> Net-(JP1-Pad2)
- OL1 pad 2: SCL -> Net-(JP2-Pad2)
- OL1 pad 3: VCC -> Net-(JP3-Pad2)
- OL1 pad 4: GND -> Net-(JP4-Pad2)
- U1 pad 11: row0 -> Net-(U1-Pad11)
- U1 pad 13: Net-(U1-Pad13) -> row0
- U1 pad 15: EncoderB -> EncoderA
- U1 pad 16: EncoderA -> EncoderB
Routing:
- net GND: track 0.00 -> 193.9 mm, vias 0 -> 2
- net Reset: track 0.00 -> 130.1 mm
- net col1: track 0.00 -> 123.5 mm
- net EncoderB: track 0.00 -> 109.3 mm
- net EncoderA: track 0.00 -> 101.4 mm
- net row1: track 0.00 -> 96.6 mm, vias 0 -> 1
- net col0: track 0.00 -> 86.5 mm
- net col2: track 0.00 -> 60.6 mm
- net row0: track 0.00 -> 59.6 mm
- net Net-(D5-Pad2): track 0.00 -> 30.2 mm
- net VCC: track 0.00 -> 26.3 mm, vias 0 -> 2
- net SDA: track 0.00 -> 24.5 mm
- net SCL: track 0.00 -> 21.0 mm
- net Net-(D2-Pad2): track 0.00 -> 14.9 mm, vias 0 -> 1
- net Net-(D1-Pad2): track 0.00 -> 14.8 mm, vias 0 -> 1
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- added copper zone on B.Cu, net GND
- added copper zone on F.Cu, net GND
Other:
- board size 136.5 x 20.6 mm -> 136.6 x 20.6 mm

Commit message: Sent for prototype
Parts:
- moved D5 1.02 mm to (163.3, 50.8)
- moved ENC1 0.95 mm to (173.0, 49.2)
- moved Reset 0.38 mm to (179.8, 51.9)
Routing:
- net GND: track 193.9 -> 174.2 mm, vias 2 -> 3
- net col1: track 123.5 -> 116.9 mm, vias 0 -> 4
- net row1: track 96.6 -> 100.9 mm
- net EncoderA: track 101.4 -> 104.0 mm
- net EncoderB: track 109.3 -> 111.8 mm
- net row0: track 59.6 -> 57.3 mm
- net Net-(D1-Pad2): track 14.8 -> 16.2 mm
- net Net-(D3-Pad2): track 14.8 -> 16.2 mm
- net Net-(D2-Pad2): track 14.9 -> 16.1 mm
- net col0: track 86.5 -> 87.3 mm, vias 0 -> 4
- net Net-(D4-Pad2): track 14.7 -> 15.4 mm
- net (no net): vias 1 -> 0

Commit message: Continued tweaks
Parts:
- D1, D2, D3, D4, D5: footprint Keebio-Parts:Diode-Hybrid-Back -> Envoy:Diode-Hybrid-Back
- MX1, MX2, MX3, MX4, MX5: footprint kbd:CherryMX_Hotswap -> Envoy:MXOnly-1U-Hotswap
- RESET1: renamed from Reset; value Reset -> SW_Push; footprint Keebio-Parts:SW_Tactile_SPST_Angled_MJTP1117-no-mount -> Envoy:Reset_Jumper_Points
- U1: footprint kbd:ProMicro_v3 -> Envoy:ProMicro_v3
- moved D3 14.2 mm to (124.9, 47.9), turned to -90 degrees
- moved D2 12.0 mm to (105.8, 51.5), turned to -90 degrees
- moved D4 12.0 mm to (143.9, 51.5), turned to -90 degrees
- moved D1 11.9 mm to (86.8, 51.5), turned to -90 degrees
- moved RESET1 1.34 mm to (179.9, 50.6), turned to -90 degrees
- moved D5 0.83 mm to (162.9, 51.5)
Connections:
- U1 pad 1: Net-(U1-Pad1) -> unconnected-(U1-Pad1)
- U1 pad 11: Net-(U1-Pad11) -> unconnected-(U1-Pad11)
- U1 pad 14: Net-(U1-Pad14) -> unconnected-(U1-Pad14)
- U1 pad 17: Net-(U1-Pad17) -> unconnected-(U1-Pad17)
- U1 pad 18: Net-(U1-Pad18) -> unconnected-(U1-Pad18)
- U1 pad 19: Net-(U1-Pad19) -> unconnected-(U1-Pad19)
- U1 pad 2: Net-(U1-Pad2) -> unconnected-(U1-Pad2)
- U1 pad 20: Net-(U1-Pad20) -> unconnected-(U1-Pad20)
- U1 pad 24: Net-(U1-Pad24) -> unconnected-(U1-Pad24)
- U1 pad 7: Net-(U1-Pad7) -> unconnected-(U1-Pad7)
Routing:
- net Net-(D5-Pad2): track 30.7 -> 19.0 mm
- net row1: track 100.9 -> 91.7 mm, vias 1 -> 0
- net row0: track 57.3 -> 48.4 mm
- net Net-(D4-Pad2): track 15.4 -> 20.7 mm
- net GND: track 174.2 -> 178.9 mm, vias 3 -> 1
- net Net-(D2-Pad2): track 16.1 -> 20.1 mm
- net Net-(D1-Pad2): track 16.2 -> 20.0 mm
- net Net-(D3-Pad2): track 16.2 -> 18.0 mm
- net Reset: track 129.8 -> 128.0 mm
- net SDA: track 24.5 -> 26.2 mm
- net EncoderA: track 104.0 -> 102.7 mm
- net col1: track 116.9 -> 116.4 mm, vias 4 -> 2
- net VCC: track 26.3 -> 26.1 mm, vias 2 -> 1
- net SCL: vias 0 -> 1
Other:
- net class Default removed
- net class Power removed
