File: piccolo-mini/piccolo-mini.sch (KiCad schematic (older format))
At the start: 13 parts, among them SW1 SW_Push, SW2 Rotary_Encoder_Switch, U1 ProMicro

Commit message: Sent for prototype
Parts:
- renumbered SW2 to ENC1, SW1 to RESET
Connections:
- net EncoderA: now also U1.13 (10/PB6); no longer U1.15 (14/PB3)
- net EncoderB: now also U1.14 (16/PB2); no longer U1.16 (15/PB1)
- net row0: now also U1.15 (14/PB3); no longer U1.13 (10/PB6)
Changed lines of the file:
@@
 $EndComp
 $Comp
-L Switch:SW_Push SW1
+L Switch:SW_Push RESET
 U 1 1 614E4310
 P 4950 1750
-F 0 "SW1" H 4950 2035 50  0000 C CNN
+F 0 "RESET" H 4950 2035 50  0000 C CNN
 F 1 "SW_Push" H 4950 1944 50  0000 C CNN
 F 2 "kbd:ResetSW_1side" H 4950 1950 50  0001 C CNN
@@
 col2
 $Comp
-L Device:Rotary_Encoder_Switch SW2
+L Device:Rotary_Encoder_Switch ENC1
 U 1 1 6150121A
 P 4750 4300
-F 0 "SW2" H 4750 4667 50  0000 C CNN
+F 0 "ENC1" H 4750 4667 50  0000 C CNN
 F 1 "Rotary_Encoder_Switch" H 4750 4576 50  0000 C CNN
 F 2 "Keebio-Parts:RotaryEncoder_EC11-no-legs" H 4600 4460 50  0001 C CNN
@@
 Text GLabel 4450 4400 0    50   Input ~ 0
 EncoderB
-Text GLabel 3050 2550 2    50   Input ~ 0
+Text GLabel 3050 2750 2    50   Input ~ 0
 EncoderA
-Text GLabel 3050 2450 2    50   Input ~ 0
+Text GLabel 3050 2650 2    50   Input ~ 0
 EncoderB
 $Comp
@@
 Wire Wire Line
 	4450 4300 3800 4300
-NoConn ~ 3050 2650
+NoConn ~ 3050 2450
 NoConn ~ 3050 2350
 NoConn ~ 3050 2250
@@
 	5300 4400 5300 3100
 Connection ~ 5300 3100
-Text GLabel 3050 2750 2    50   Input ~ 0
+Text GLabel 3050 2550 2    50   Input ~ 0
 row0
 NoConn ~ 1650 2650
