File: piccolo/piccolo-backplate/piccolo-backplate.kicad_pcb (KiCad board)
At the start: 2 copper layers, 136.6 x 20.6 mm, 3 parts

Commit message: Logo added to backplate
Parts:
- added G***: LOGO, Envoy:Piccolo_Macro_Pad_text_30mm, B.Cu at (175.6, 99.8)
- added G***: LOGO, Envoy:piccolo_logo_100mm, B.Cu at (142.2, 93.5)
