File: piccolo/piccolo-backplate/piccolo-backplate.kicad_pcb (KiCad board)
At the start: 2 copper layers, 136.6 x 20.6 mm, 9 parts

Commit message: Add identifiers to boards
Other:
- board text added: "Piccolo Macro Pad Backplate by JeJeff rev 0.2"
Changed lines of the file:
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@@
       ) (layer "B.SilkS") (width 0) (fill solid))
   )
+  (gr_line (start 73.15 104.7) (end 209.8 84.05) (layer "Dwgs.User") (width 0.15))
+  (gr_line (start 209.8 104.7) (end 73.2 84.1) (layer "Dwgs.User") (width 0.15))
   (gr_arc (start 73.979118 84.846655) (end 73.979118 84.052905) (angle -90) (layer "Edge.Cuts") (width 0.05))
   (gr_line (start 73.979118 104.690405) (end 209.011868 104.690405) (layer "Edge.Cuts") (width 0.05))
@@
     (effects (font (size 0.8 0.8) (thickness 0.15)))
   )
+  (gr_text "Piccolo Macro Pad Backplate\nby JeJeff\nrev 0.2" (at 141.45 94.35) (layer "F.Mask")
+    (effects (font (size 1 1) (thickness 0.2)))
+  )
   (dimension (type aligned) (layer "Dwgs.User")

Commit message: make oled cutout larger in switchplate.  Prepare rev3 gerbers
Parts:
- G***: footprint Envoy:piccolo_logo_100mm -> Envoy:piccolo_logo_100mm_mask
Other:
- board text added: "Piccolo Macro Pad Backplate by JeJeff rev 0.3"
- board text removed: "Piccolo Macro Pad Backplate by JeJeff rev 0.2"
