File: piccolo/piccolo-switchplate/piccolo-switchplate.kicad_pcb (KiCad board)
At the start: 2 copper layers, 136.6 x 20.6 mm, 9 parts

Commit message: Sent switchplate to PCB manufacturer for first prototype.
Parts:
- added ENC1: Rotary_Encoder_Switch, Envoy:RotaryEncoder_Cutout, F.Cu at (195.4, 118.3)
Other:
- board text added: "JLCJLCJLCJLC"
Changed lines of the file:
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@@
       (layerselection 0x00010fc_ffffffff)
       (disableapertmacros false)
-      (usegerberextensions false)
+      (usegerberextensions true)
       (usegerberattributes true)
       (usegerberadvancedattributes true)
@@
       (outputformat 1)
       (mirror false)
-      (drillshape 1)
+      (drillshape 0)
       (scaleselection 1)
-      (outputdirectory "")
+      (outputdirectory "gerbers")
     )
   )
@@
     (pad "" np_thru_hole oval (at 0 6.75) (size 14 0.5) (drill oval 14 0.5) (layers *.Cu *.Mask))
   )
+  (footprint "Envoy:RotaryEncoder_Cutout" (layer "F.Cu")
+    (at 195.387496 118.3125 90)
+    (descr "Alps rotary encoder, EC12E... with switch, vertical shaft, http://www.alps.com/prod/info/E/HTML/Encoder/Incremental/EC11/EC11E15204A3.html")
+    (tags "rotary encoder")
+    (property "Sheetfile" "piccolo-switchplate.kicad_sch")
+    (property "Sheetname" "")
+    (fp_text reference "ENC1" (at 0.0635 0.03175 90) (layer "F.SilkS") hide
+      (effects (font (size 1 1) (thickness 0.15)))
+    )
+    (fp_text value "Rotary_Encoder_Switch" (at 0 7.9 90) (layer "F.Fab")
+      (effects (font (size 1 1) (thickness 0.15)))
+    )
+    (fp_text user "${REFERENCE}" (at 3.6 3.8 90) (layer "F.Fab")
+      (effects (font (size 1 1) (thickness 0.15)))
+    )
+    (fp_line (start -9 -7.1) (end -9 7.1) (layer "F.CrtYd") (width 0.05))
+    (fp_line (start 8.5 7.1) (end -9 7.1) (layer "F.CrtYd") (width 0.05))
+    (fp_line (start 8.5 7.1) (end 8.5 -7.1) (layer "F.CrtYd") (width 0.05))
+    (fp_line (start -9 -7.1) (end 8.5 -7.1) (layer "F.CrtYd") (width 0.05))
+    (fp_line (start 6 5.8) (end -6 5.8) (layer "F.Fab") (width 0.12))
+    (pad "" np_thru_hole oval (at 6.85 0 90) (size 0.5 12) (drill oval 0.5 12) (layers *.Cu *.Mask))
+    (pad "" np_thru_hole oval (at -6.85 0 90) (size 0.5 12) (drill oval 0.5 12) (layers *.Cu *.Mask))
+    (pad "" np_thru_hole oval (at 0 5.75 90) (size 14.2 0.5) (drill oval 14.2 0.5) (layers *.Cu *.Mask))
+    (pad "" np_thru_hole oval (at 0 -5.75 90) (size 14.2 0.5) (drill oval 14.2 0.5) (layers *.Cu *.Mask))
+    (model "${KISYS3DMOD}/Rotary_Encoder.3dshapes/RotaryEncoder_Alps_EC11E-Switch_Vertical_H20mm.wrl"
+      (offset (xyz 0 0 0))
+      (scale (xyz 1 1 1))
+      (rotate (xyz 0 0 0))
+    )
+  )
   (footprint "Envoy:MountingHole_Reinforced_2.5mm" (layer "F.Cu")
     (at 109.662496 111.16875)
@@
   (gr_arc (start 69.879746 127.8375) (end 69.085996 127.8375) (angle -90) (layer "Edge.Cuts") (width 0.05))
   (gr_arc (start 204.912496 127.8375) (end 204.912496 128.63125) (angle -90) (layer "Edge.Cuts") (width 0.05))
+  (gr_text "JLCJLCJLCJLC" (at 128.5875 119.0625 90) (layer "B.SilkS")
+    (effects (font (size 0.8 0.8) (thickness 0.15)) (justify mirror))
+  )
   (dimension (type aligned) (layer "Dwgs.User")
     (pts (xy 204.912496 128.63125) (xy 204.912496 107.99375))

Commit message: Add identifiers to boards
Other:
- board text added: "Piccolo Macro Pad Switchplate by JeJeff rev 0.2"
Changed lines of the file:
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@@
   (setup
     (pad_to_mask_clearance 0)
+    (grid_origin 119.187496 118.3125)
     (pcbplotparams
       (layerselection 0x00010fc_ffffffff)
@@
     (effects (font (size 0.8 0.8) (thickness 0.15)) (justify mirror))
   )
+  (gr_text "Piccolo Macro Pad\nSwitchplate\nby JeJeff\nrev 0.2" (at 107.087496 118.5625 90) (layer "B.Mask")
+    (effects (font (size 1 1) (thickness 0.2)) (justify mirror))
+  )
   (dimension (type aligned) (layer "Dwgs.User")

Commit message: make oled cutout larger in switchplate.  Prepare rev3 gerbers
Other:
- board text added: "Piccolo Macro Pad Switchplate by JeJeff rev 0.3"
- board text removed: "Piccolo Macro Pad Switchplate by JeJeff rev 0.2"
Changed lines of the file:
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@@
     (property "Sheetfile" "piccolo-switchplate.kicad_sch")
     (property "Sheetname" "")
+    (attr through_hole)
     (fp_text reference "MX4" (at 0.25 10.05) (layer "Eco2.User") hide
       (effects (font (size 1 1) (thickness 0.15)))
@@
       (effects (font (size 1 1) (thickness 0.15)))
     )
-    (fp_line (start 9.5 -9.5) (end 9.5 9.5) (layer "Dwgs.User") (width 0.15))
-    (fp_line (start -9.5 9.5) (end -9.5 -9.5) (layer "Dwgs.User") (width 0.15))
-    (fp_line (start 9.5 9.5) (end -9.5 9.5) (layer "Dwgs.User") (width 0.15))
-    (fp_line (start -9.5 -9.5) (end 9.5 -9.5) (layer "Dwgs.User") (width 0.15))
-    (pad "" np_thru_hole oval (at 0 6.75) (size 14 0.5) (drill oval 14 0.5) (layers *.Cu *.Mask))
-    (pad "" np_thru_hole oval (at 0 -6.75) (size 14 0.5) (drill oval 14 0.5) (layers *.Cu *.Mask))
-    (pad "" np_thru_hole oval (at 6.75 0) (size 0.5 14) (drill oval 0.5 14) (layers *.Cu *.Mask))
-    (pad "" np_thru_hole oval (at -6.75 0) (size 0.5 14) (drill oval 0.5 14) (layers *.Cu *.Mask))
+    (fp_line (start -9.5 -9.5) (end 9.5 -9.5) (layer "Dwgs.User") (width 0.15))
+    (fp_line (start 9.5 -9.5) (end 9.5 9.5) (layer "Dwgs.User") (width 0.15))
+    (fp_line (start 9.5 9.5) (end -9.5 9.5) (layer "Dwgs.User") (width 0.15))
+    (fp_line (start -9.5 9.5) (end -9.5 -9.5) (layer "Dwgs.User") (width 0.15))
+    (fp_line (start 7 7) (end 7 -7) (layer "Cmts.User") (width 0.12))
+    (fp_line (start -7 7) (end 7 7) (layer "Cmts.User") (width 0.12))
+    (fp_line (start -7 7) (end -7 -7) (layer "Cmts.User") (width 0.12))
+    (fp_line (start -7 -7) (end 7 -7) (layer "Cmts.User") (width 0.12))
+    (fp_rect (start -7 -7) (end 7 7) (layer "Edge.Cuts") (width 0.1) (fill none))
   )
   (footprint "Envoy:MountingHole_Reinforced_2.5mm" (layer "F.Cu")
@@
     (fp_rect (start 6 -33.5) (end 5.75 -33.25) (layer "Cmts.User") (width 0.12) (fill none))
     (fp_rect (start -6 -33.5) (end -5.75 -33.25) (layer "Cmts.User") (width 0.12) (fill none))
-    (fp_rect (start 5.74 -3.75) (end -5.75 -33.25) (layer "Edge.Cuts") (width 0.12) (fill none))
+    (fp_rect (start 5.85 -3.45) (end -5.86 -33.25) (layer "Edge.Cuts") (width 0.12) (fill none))
   )
   (footprint "Envoy:MX_Switch_Cutout_Square" (layer "F.Cu")
@@
     (property "Sheetfile" "piccolo-switchplate.kicad_sch")
     (property "Sheetname" "")
+    (attr through_hole)
     (fp_text reference "MX1" (at 0.25 10.05) (layer "Eco2.User") hide
       (effects (font (size 1 1) (thickness 0.15)))
@@
       (effects (font (size 1 1) (thickness 0.15)))
     )
-    (fp_line (start -9.5 9.5) (end -9.5 -9.5) (layer "Dwgs.User") (width 0.15))
-    (fp_line (start 9.5 -9.5) (end 9.5 9.5) (layer "Dwgs.User") (width 0.15))
-    (fp_line (start -9.5 -9.5) (end 9.5 -9.5) (layer "Dwgs.User") (width 0.15))
-    (fp_line (start 9.5 9.5) (end -9.5 9.5) (layer "Dwgs.User") (width 0.15))
-    (pad "" np_thru_hole oval (at -6.75 0) (size 0.5 14) (drill oval 0.5 14) (layers *.Cu *.Mask))
-    (pad "" np_thru_hole oval (at 0 -6.75) (size 14 0.5) (drill oval 14 0.5) (layers *.Cu *.Mask))
-    (pad "" np_thru_hole oval (at 6.75 0) (size 0.5 14) (drill oval 0.5 14) (layers *.Cu *.Mask))
-    (pad "" np_thru_hole oval (at 0 6.75) (size 14 0.5) (drill oval 14 0.5) (layers *.Cu *.Mask))
+    (fp_line (start 9.5 -9.5) (end 9.5 9.5) (layer "Dwgs.User") (width 0.15))
+    (fp_line (start -9.5 9.5) (end -9.5 -9.5) (layer "Dwgs.User") (width 0.15))
+    (fp_line (start -9.5 -9.5) (end 9.5 -9.5) (layer "Dwgs.User") (width 0.15))
+    (fp_line (start 9.5 9.5) (end -9.5 9.5) (layer "Dwgs.User") (width 0.15))
+    (fp_line (start -7 7) (end -7 -7) (layer "Cmts.User") (width 0.12))
+    (fp_line (start -7 7) (end 7 7) (layer "Cmts.User") (width 0.12))
+    (fp_line (start 7 7) (end 7 -7) (layer "Cmts.User") (width 0.12))
+    (fp_line (start -7 -7) (end 7 -7) (layer "Cmts.User") (width 0.12))
+    (fp_rect (start -7 -7) (end 7 7) (layer "Edge.Cuts") (width 0.1) (fill none))
   )
   (footprint "Envoy:MX_Switch_Cutout_Square" (layer "F.Cu")
@@
     (property "Sheetfile" "piccolo-switchplate.kicad_sch")
     (property "Sheetname" "")
+    (attr through_hole)
     (fp_text reference "MX3" (at 0.25 10.05) (layer "Eco2.User") hide
       (effects (font (size 1 1) (thickness 0.15)))
@@
       (effects (font (size 1 1) (thickness 0.15)))
     )
-    (fp_line (start -9.5 -9.5) (end 9.5 -9.5) (layer "Dwgs.User") (width 0.15))
-    (fp_line (start 9.5 9.5) (end -9.5 9.5) (layer "Dwgs.User") (width 0.15))
-    (fp_line (start -9.5 9.5) (end -9.5 -9.5) (layer "Dwgs.User") (width 0.15))
-    (fp_line (start 9.5 -9.5) (end 9.5 9.5) (layer "Dwgs.User") (width 0.15))
-    (pad "" np_thru_hole oval (at 0 -6.75) (size 14 0.5) (drill oval 14 0.5) (layers *.Cu *.Mask))
-    (pad "" np_thru_hole oval (at 6.75 0) (size 0.5 14) (drill oval 0.5 14) (layers *.Cu *.Mask))
-    (pad "" np_thru_hole oval (at -6.75 0) (size 0.5 14) (drill oval 0.5 14) (layers *.Cu *.Mask))
-    (pad "" np_thru_hole oval (at 0 6.75) (size 14 0.5) (drill oval 14 0.5) (layers *.Cu *.Mask))
+    (fp_line (start 9.5 -9.5) (end 9.5 9.5) (layer "Dwgs.User") (width 0.15))
+    (fp_line (start -9.5 -9.5) (end 9.5 -9.5) (layer "Dwgs.User") (width 0.15))
+    (fp_line (start 9.5 9.5) (end -9.5 9.5) (layer "Dwgs.User") (width 0.15))
+    (fp_line (start -9.5 9.5) (end -9.5 -9.5) (layer "Dwgs.User") (width 0.15))
+    (fp_line (start 7 7) (end 7 -7) (layer "Cmts.User") (width 0.12))
+    (fp_line (start -7 7) (end 7 7) (layer "Cmts.User") (width 0.12))
+    (fp_line (start -7 7) (end -7 -7) (layer "Cmts.User") (width 0.12))
+    (fp_line (start -7 -7) (end 7 -7) (layer "Cmts.User") (width 0.12))
+    (fp_rect (start -7 -7) (end 7 7) (layer "Edge.Cuts") (width 0.1) (fill none))
   )
   (footprint "Envoy:MX_Switch_Cutout_Square" (layer "F.Cu")
@@
     (property "Sheetfile" "piccolo-switchplate.kicad_sch")
     (property "Sheetname" "")
+    (attr through_hole)
     (fp_text reference "MX2" (at 0.25 10.05) (layer "Eco2.User") hide
       (effects (font (size 1 1) (thickness 0.15)))
@@
       (effects (font (size 1 1) (thickness 0.15)))
     )
-    (fp_line (start 9.5 9.5) (end -9.5 9.5) (layer "Dwgs.User") (width 0.15))
-    (fp_line (start 9.5 -9.5) (end 9.5 9.5) (layer "Dwgs.User") (width 0.15))
-    (fp_line (start -9.5 -9.5) (end 9.5 -9.5) (layer "Dwgs.User") (width 0.15))
-    (fp_line (start -9.5 9.5) (end -9.5 -9.5) (layer "Dwgs.User") (width 0.15))
-    (pad "" np_thru_hole oval (at -6.75 0) (size 0.5 14) (drill oval 0.5 14) (layers *.Cu *.Mask))
-    (pad "" np_thru_hole oval (at 6.75 0) (size 0.5 14) (drill oval 0.5 14) (layers *.Cu *.Mask))
-    (pad "" np_thru_hole oval (at 0 -6.75) (size 14 0.5) (drill oval 14 0.5) (layers *.Cu *.Mask))
-    (pad "" np_thru_hole oval (at 0 6.75) (size 14 0.5) (drill oval 14 0.5) (layers *.Cu *.Mask))
+    (fp_line (start -9.5 9.5) (end -9.5 -9.5) (layer "Dwgs.User") (width 0.15))
+    (fp_line (start 9.5 -9.5) (end 9.5 9.5) (layer "Dwgs.User") (width 0.15))
+    (fp_line (start 9.5 9.5) (end -9.5 9.5) (layer "Dwgs.User") (width 0.15))
+    (fp_line (start -9.5 -9.5) (end 9.5 -9.5) (layer "Dwgs.User") (width 0.15))
+    (fp_line (start 7 7) (end 7 -7) (layer "Cmts.User") (width 0.12))
+    (fp_line (start -7 7) (end -7 -7) (layer "Cmts.User") (width 0.12))
+    (fp_line (start -7 -7) (end 7 -7) (layer "Cmts.User") (width 0.12))
+    (fp_line (start -7 7) (end 7 7) (layer "Cmts.User") (width 0.12))
+    (fp_rect (start -7 -7) (end 7 7) (layer "Edge.Cuts") (width 0.1) (fill none))
   )
   (footprint "Envoy:MX_Switch_Cutout_Square" (layer "F.Cu")
@@
     (property "Sheetfile" "piccolo-switchplate.kicad_sch")
     (property "Sheetname" "")
+    (attr through_hole)
     (fp_text reference "MX5" (at 0.25 10.05) (layer "Eco2.User") hide
       (effects (font (size 1 1) (thickness 0.15)))
@@
     (fp_line (start 9.5 9.5) (end -9.5 9.5) (layer "Dwgs.User") (width 0.15))
     (fp_line (start -9.5 -9.5) (end 9.5 -9.5) (layer "Dwgs.User") (width 0.15))
-    (fp_line (start 9.5 -9.5) (end 9.5 9.5) (layer "Dwgs.User") (width 0.15))
-    (fp_line (start -9.5 9.5) (end -9.5 -9.5) (layer "Dwgs.User") (width 0.15))
-    (pad "" np_thru_hole oval (at 0 -6.75) (size 14 0.5) (drill oval 14 0.5) (layers *.Cu *.Mask))
-    (pad "" np_thru_hole oval (at -6.75 0) (size 0.5 14) (drill oval 0.5 14) (layers *.Cu *.Mask))
-    (pad "" np_thru_hole oval (at 6.75 0) (size 0.5 14) (drill oval 0.5 14) (layers *.Cu *.Mask))
-    (pad "" np_thru_hole oval (at 0 6.75) (size 14 0.5) (drill oval 14 0.5) (layers *.Cu *.Mask))
+    (fp_line (start -9.5 9.5) (end -9.5 -9.5) (layer "Dwgs.User") (width 0.15))
+    (fp_line (start 9.5 -9.5) (end 9.5 9.5) (layer "Dwgs.User") (width 0.15))
+    (fp_line (start 7 7) (end 7 -7) (layer "Cmts.User") (width 0.12))
+    (fp_line (start -7 7) (end 7 7) (layer "Cmts.User") (width 0.12))
+    (fp_line (start -7 -7) (end 7 -7) (layer "Cmts.User") (width 0.12))
+    (fp_line (start -7 7) (end -7 -7) (layer "Cmts.User") (width 0.12))
+    (fp_rect (start -7 -7) (end 7 7) (layer "Edge.Cuts") (width 0.1) (fill none))
   )
   (footprint "Envoy:RotaryEncoder_Cutout" (layer "F.Cu")
@@
     (effects (font (size 0.8 0.8) (thickness 0.15)) (justify mirror))
   )
-  (gr_text "Piccolo Macro Pad\nSwitchplate\nby JeJeff\nrev 0.2" (at 107.087496 118.5625 90) (layer "B.Mask")
+  (gr_text "Piccolo Macro Pad\nSwitchplate\nby JeJeff\nrev 0.3" (at 107.087496 118.5625 90) (layer "B.Mask")
     (effects (font (size 1 1) (thickness 0.2)) (justify mirror))
   )

Commit message: Made the oled cutout larger. because the pins interfere with the switchplate.  Bump rev to 0.4
Other:
- board text added: "Piccolo Macro Pad Switchplate by JeJeff rev 0.4"
- board text removed: "Piccolo Macro Pad Switchplate by JeJeff rev 0.3"
Changed lines of the file:
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@@
     (fp_rect (start 6 -33.5) (end 5.75 -33.25) (layer "Cmts.User") (width 0.12) (fill none))
     (fp_rect (start -6 -33.5) (end -5.75 -33.25) (layer "Cmts.User") (width 0.12) (fill none))
-    (fp_rect (start 5.85 -3.45) (end -5.86 -33.25) (layer "Edge.Cuts") (width 0.12) (fill none))
+    (fp_rect (start 5.85 1.12) (end -5.86 -33.5) (layer "Edge.Cuts") (width 0.12) (fill none))
   )
   (footprint "Envoy:MX_Switch_Cutout_Square" (layer "F.Cu")
@@
     (effects (font (size 0.8 0.8) (thickness 0.15)) (justify mirror))
   )
-  (gr_text "Piccolo Macro Pad\nSwitchplate\nby JeJeff\nrev 0.3" (at 107.087496 118.5625 90) (layer "B.Mask")
-    (effects (font (size 1 1) (thickness 0.2)) (justify mirror))
+  (gr_text "Piccolo Macro Pad Switchplate\nby JeJeff rev 0.4" (at 89.187496 110.1125) (layer "B.Mask")
+    (effects (font (size 1 1) (thickness 0.25)) (justify mirror))
   )
   (dimension (type aligned) (layer "Dwgs.User")
